File: PowerNode/Power Node V2.0/PowerNode2.sch (KiCad schematic (older format))
At the start: 34 parts, among them IC2 7449N, IC3 7449N, IC4 ACS712-LC, IC5 74595N, IC6 741G04DBV

Commit message: Fixed a library renaming issue
Parts:
- C1, C2, C3: symbol PowerNode2-eagle-import:C5_3 -> PowerNode2:C5_3
- CURR1, PWRLED1, VOLT1: symbol PowerNode2-eagle-import:LED5MM -> PowerNode2:LED5MM
- DP1, PB2, QH*1: symbol PowerNode2-eagle-import:2,54_0,9 -> PowerNode2:2,54_0,9
- GND1, GND2: symbol PowerNode2-eagle-import:2,15_1,0 -> PowerNode2:2,15_1,0
- GND3, SCL1, SDA1, VCC1: symbol PowerNode2-eagle-import:WIREPAD1,6_0,9 -> PowerNode2:WIREPAD1,6_0,9
- GNDHIIN1, GNDHIOUT1, VHIIN1, VHIOUT1: symbol PowerNode2-eagle-import:WIREPAD4,16O1,6 -> PowerNode2:WIREPAD4,16O1,6
- IC2, IC3: symbol PowerNode2-eagle-import:7449N -> PowerNode2:7449N
- IC4: symbol PowerNode2-eagle-import:ACS712-LC -> PowerNode2:ACS712-LC
- IC5: symbol PowerNode2-eagle-import:74595N -> PowerNode2:74595N
- IC6: symbol PowerNode2-eagle-import:741G04DBV -> PowerNode2:741G04DBV
- LED1, LED2: symbol PowerNode2-eagle-import:S4301B -> PowerNode2:S4301B
- R1, R2, R4, R5, R6: symbol PowerNode2-eagle-import:R-US_0411_15 -> PowerNode2:R-US_0411_15
- R3: symbol PowerNode2-eagle-import:TRIM_US-B25P -> PowerNode2:TRIM_US-B25P
- S1: symbol PowerNode2-eagle-import:TL32PO -> PowerNode2:TL32PO
- U$1: symbol PowerNode2-eagle-import:ATTINY84ATTINY84-20PU -> PowerNode2:ATTINY84ATTINY84-20PU
Changed lines of the file:
@@
 Connection ~ 5600 6300
 $Comp
-L PowerNode2-eagle-import:ATTINY84ATTINY84-20PU U$1
+L PowerNode2:ATTINY84ATTINY84-20PU U$1
 U 1 1 BABD3B23
 P 3700 3700
@@
 $EndComp
 $Comp
-L PowerNode2-eagle-import:C5_3 C1
+L PowerNode2:C5_3 C1
 U 1 1 DB2CE5A6
 P 6900 5900
@@
 $EndComp
 $Comp
-L PowerNode2-eagle-import:C5_3 C2
+L PowerNode2:C5_3 C2
 U 1 1 B94C3227
 P 1300 2800
@@
 $EndComp
 $Comp
-L PowerNode2-eagle-import:WIREPAD1,6_0,9 VCC1
+L PowerNode2:WIREPAD1,6_0,9 VCC1
 U 1 1 D0DD1D8E
 P 800 2700
@@
 $EndComp
 $Comp
-L PowerNode2-eagle-import:WIREPAD1,6_0,9 GND3
+L PowerNode2:WIREPAD1,6_0,9 GND3
 U 1 1 8E097FD0
 P 800 3000
@@
 $EndComp
 $Comp
-L PowerNode2-eagle-import:WIREPAD1,6_0,9 SDA1
+L PowerNode2:WIREPAD1,6_0,9 SDA1
 U 1 1 943CED1C
 P 5100 3700
@@
 $EndComp
 $Comp
-L PowerNode2-eagle-import:WIREPAD1,6_0,9 SCL1
+L PowerNode2:WIREPAD1,6_0,9 SCL1
 U 1 1 252148C1
 P 5100 3900
@@
 $EndComp
 $Comp
-L PowerNode2-eagle-import:R-US_0411_15 R1
+L PowerNode2:R-US_0411_15 R1
 U 1 1 6C31DF7B
 P 3400 2500
@@
 $EndComp
 $Comp
-L PowerNode2-eagle-import:R-US_0411_15 R2
+L PowerNode2:R-US_0411_15 R2
 U 1 1 00509794
 P 4100 2500
@@
 $EndComp
 $Comp
-L PowerNode2-eagle-import:WIREPAD4,16O1,6 VHIIN1
+L PowerNode2:WIREPAD4,16O1,6 VHIIN1
 U 1 1 3ABF0FC0
 P 6300 2500
@@
 $EndComp
 $Comp
-L PowerNode2-eagle-import:TRIM_US-B25P R3
+L PowerNode2:TRIM_US-B25P R3
 U 1 1 9D3B2993
 P 6300 3800
@@
 $EndComp
 $Comp
-L PowerNode2-eagle-import:WIREPAD4,16O1,6 GNDHIIN1
+L PowerNode2:WIREPAD4,16O1,6 GNDHIIN1
 U 1 1 9FE8900C
 P 1400 4300
@@
 $EndComp
 $Comp
-L PowerNode2-eagle-import:S4301B LED1
+L PowerNode2:S4301B LED1
 U 1 1 D5D4A691
 P 9600 3400
@@
 $EndComp
 $Comp
-L PowerNode2-eagle-import:S4301B LED2
+L PowerNode2:S4301B LED2
 U 1 1 6A31474D
 P 9600 4500
@@
 $EndComp
 $Comp
-L PowerNode2-eagle-import:7449N IC2
+L PowerNode2:7449N IC2
 U 1 1 541775CA
 P 8700 3400
@@
 $EndComp
 $Comp
-L PowerNode2-eagle-import:7449N IC3
+L PowerNode2:7449N IC3
 U 1 1 5ED25CA7
 P 8700 4500
@@
 $EndComp
 $Comp
-L PowerNode2-eagle-import:7449N IC2
+L PowerNode2:7449N IC2
 U 2 1 541775C6
 P 1700 1700
@@
 $EndComp
 $Comp
-L PowerNode2-eagle-import:7449N IC3
+L PowerNode2:7449N IC3
 U 2 1 5ED25CAB
 P 2200 1700
@@
 $EndComp
 $Comp
-L PowerNode2-eagle-import:ACS712-LC IC4
+L PowerNode2:ACS712-LC IC4
 U 1 1 46657C43
 P 5700 5600
@@
 $EndComp
 $Comp
-L PowerNode2-eagle-import:74595N IC5
+L PowerNode2:74595N IC5
 U 1 1 E57833A7
 P 7200 3600
@@
 $EndComp
 $Comp
-L PowerNode2-eagle-import:C5_3 C3
+L PowerNode2:C5_3 C3
 U 1 1 DAA3AADF
 P 5900 4400
@@
 $EndComp
 $Comp
-L PowerNode2-eagle-import:74595N IC5
+L PowerNode2:74595N IC5
 U 2 1 E57833AB
 P 2700 1700
@@
 $EndComp
 $Comp
-L PowerNode2-eagle-import:LED5MM PWRLED1
+L PowerNode2:LED5MM PWRLED1
 U 1 1 EEAA4052
 P 2200 3000
@@
 $EndComp
 $Comp
-L PowerNode2-eagle-import:R-US_0411_15 R4
+L PowerNode2:R-US_0411_15 R4
 U 1 1 F98F597E
 P 2200 3500
@@
 $EndComp
 $Comp
-L PowerNode2-eagle-import:EAGLE-TOP-15MM #LOGO1
+L PowerNode2:EAGLE-TOP-15MM #LOGO1
 U 1 1 8712EDD9
 P 1200 5600
@@
 $EndComp
 $Comp
-L PowerNode2-eagle-import:TL32PO S1
+L PowerNode2:TL32PO S1
 U 1 1 CEBFFD5E
 P 6800 2200
@@
 $EndComp
 $Comp
-L PowerNode2-eagle-import:LED5MM CURR1
+L PowerNode2:LED5MM CURR1
 U 1 1 46B498CE
 P 8400 2200
@@
 $EndComp
 $Comp
-L PowerNode2-eagle-import:R-US_0411_15 R5
+L PowerNode2:R-US_0411_15 R5
 U 1 1 6637B0E6
 P 8900 2200
@@
 $EndComp
 $Comp
-L PowerNode2-eagle-import:LED5MM VOLT1
+L PowerNode2:LED5MM VOLT1
 U 1 1 24952B63
 P 8400 2600
@@
 $EndComp
 $Comp
-L PowerNode2-eagle-import:R-US_0411_15 R6
+L PowerNode2:R-US_0411_15 R6
 U 1 1 F7B4B2BB
 P 8900 2600
@@
 $EndComp
 $Comp
-L PowerNode2-eagle-import:741G04DBV IC6
+L PowerNode2:741G04DBV IC6
 U 1 1 6A4BA564
 P 7800 2200
@@
 $EndComp
 $Comp
-L PowerNode2-eagle-import:741G04DBV IC6
+L PowerNode2:741G04DBV IC6
 U 2 1 6A4BA568
 P 1400 1700
@@
 $EndComp
 $Comp
-L PowerNode2-eagle-import:2,54_0,9 PB2
+L PowerNode2:2,54_0,9 PB2
 U 1 1 F1E52EE7
 P 5000 3200
@@
 $EndComp
 $Comp
-L PowerNode2-eagle-import:2,54_0,9 QH*1
+L PowerNode2:2,54_0,9 QH*1
 U 1 1 2C9469AA
 P 7600 4500
@@
 $EndComp
 $Comp
-L PowerNode2-eagle-import:2,54_0,9 DP1
+L PowerNode2:2,54_0,9 DP1
 U 1 1 2762D014
 P 11100 4200
@@
 $EndComp
 $Comp
-L PowerNode2-eagle-import:2,15_1,0 GND1
+L PowerNode2:2,15_1,0 GND1
 U 1 1 DB8695AC
 P 1500 3200
@@
 $EndComp
 $Comp
-L PowerNode2-eagle-import:2,15_1,0 GND2
+L PowerNode2:2,15_1,0 GND2
 U 1 1 13A376EC
 P 1500 3400
@@
 $EndComp
 $Comp
-L PowerNode2-eagle-import:WIREPAD4,16O1,6 GNDHIOUT1
+L PowerNode2:WIREPAD4,16O1,6 GNDHIOUT1
 U 1 1 16E6194B
 P 5600 6700
@@
 $EndComp
 $Comp
-L PowerNode2-eagle-import:WIREPAD4,16O1,6 VHIOUT1
+L PowerNode2:WIREPAD4,16O1,6 VHIOUT1
 U 1 1 8575F09C
 P 5700 2300
